File: kicad/isl94202.sch (KiCad schematic (older format))
At the start: 93 parts, among them Q1 NDS0605, Q15 BSS138, Q2 NDS0605, Q3 NDS0605, Q4 BSS138, Q5 BSS138, Q6 BSS138, Q7 BSS138, Q8 BSS138, Q9 NDS0605, U7 ISL94202

Commit message: Fix issues found during testing (v0.1.1)
- Add BAT+/- and EXT+/- markings to terminals (#2)
- Change C30 to 470nF (#5)
- Add C20 (47nF) at VC0 pin (#5)
- Add C21 and R72 for proper low-pass filter of VDD (#5)
- Change C39 at VREF to 1uF (#5)
- Add R70: Pull-down for PCHG FET (#5)
- Add R73: Weak pull-down for 5V supply (#6)
Parts:
- removed JP3, JP4: 7, Jumper:SolderJumper-2_P1.3mm_Open_RoundedPad1.0x1.5mm, symbol Jumper:SolderJumper_2_Open
- removed R73, R74, R75, R77, R78, R79, R80, R81, R82, R83: 0R, LibreSolar:R_0603_1608, symbol Project:R
- added C20: 47n, LibreSolar:C_0603_1608, symbol Project:C
- added C21: 4.7u, LibreSolar:C_1206_3216, symbol Project:C
- C30: value 47n -> 470n; Manufacturer Yageo -> (none); PartNumber CC0603KRX7R9BB473 -> (none)
- C39: value 100n -> 1u; Manufacturer Yageo -> (none); PartNumber CC0603KRX7R9BB104 -> (none)
- R72: value 0R -> 4R7; PartNumber RC0603FR-070RL -> RC0603FR-071KL
Connections:
- net labels added: TEMPO
- net labels removed: TEMP0
- wire segments 288 -> 268
Other:
- note removed: "3 cells"
- note removed: "3/4 cells"
- note removed: "3/4/5 cells"
- note removed: "3/4/5/6 cells"
- note removed: "3/4/5/6/7 cells"
- moved on the sheet: D2

Commit message: Update to v0.2
- Switch to STM32L452 MCU (STM32F072 has too little RAM for CAN ISO-TP etc.)
- Add CAN termination jumper
- Add CAN bus power supply diodes
- Update CAN connector to match LS.bus spec
- Add interactive BOM and CSV BOM to build directory
- Add additional thermal vias with 0.2mm diameter under MOSFETs
Changed lines of the file:
@@
 Sheet 5 5
 Title "BMS 8S50 IC"
-Date "2020-05-08"
-Rev "0.1.1"
-Comp "Libre Solar"
-Comment1 ""
-Comment2 ""
-Comment3 ""
+Date "2021-02-13"
+Rev "0.2"
+Comp "Libre Solar Technologies GmbH"
+Comment1 "Website: https://libre.solar"
+Comment2 "Author: Martin Jäger"
+Comment3 "License: Creative Commons Attribution-ShareAlike 4.0 International"
 Comment4 ""
 $EndDescr
@@
 	6100 1300 6100 1100
 Wire Wire Line
-	6100 1100 5500 1100
+	6100 1100 5800 1100
 Wire Wire Line
 	5500 1100 5500 1400
@@
 Wire Wire Line
 	4800 1400 5500 1400
+$Comp
+L power:PWR_FLAG #FLG0102
+U 1 1 6053486C
+P 5800 1000
+F 0 "#FLG0102" H 5800 1075 50  0001 C CNN
+F 1 "PWR_FLAG" H 5800 1173 50  0000 C CNN
+F 2 "" H 5800 1000 50  0001 C CNN
+F 3 "~" H 5800 1000 50  0001 C CNN
+	1    5800 1000
+	1    0    0    -1
+$EndComp
+Wire Wire Line
+	5800 1100 5800 1000
+Connection ~ 5800 1100
+Wire Wire Line
+	5800 1100 5500 1100
 $EndSCHEMATC
