File: kicad/mcu.sch (KiCad schematic (older format))
At the start: 24 parts, among them P5 CONN_01X02, U2 TCAN334, U3 STM32F072CBU6, U6 24AA32, Y1 8MHz

Commit message: Update to v0.2
- Switch to STM32L452 MCU (STM32F072 has too little RAM for CAN ISO-TP etc.)
- Add CAN termination jumper
- Add CAN bus power supply diodes
- Update CAN connector to match LS.bus spec
- Add interactive BOM and CSV BOM to build directory
- Add additional thermal vias with 0.2mm diameter under MOSFETs
Parts:
- added JP3: Jumper_NC_Small, Connector_PinHeader_2.54mm:PinHeader_1x02_P2.54mm_Vertical, symbol Device:Jumper_NC_Small
- U3: value STM32F072CBU6 -> STM32L452CCU6; symbol MCU_ST_STM32F0:STM32F072CBUx -> MCU_ST_STM32L4:STM32L452CCUx; PartNumber STM32F072CBU6 -> STM32L452CCU6
- U6: symbol LibreSolar:24AA01 -> LibreSolar:24AAxx-OT
Connections:
- net CAN_H: now also JP3.1; no longer R69.1
- new net: JP3.2, R69.1
Other:
- note added: "MCU STM32L452"
- note removed: "Alternative: STM32L452CxU6"
- note removed: "MCU STM32F072"
- note removed: "TODO!!!\nBQ769x0 ID either 0x08 or 0x18\n24AA01 has 0b1010XXX --> OK"
- moved on the sheet: C27, C31, R35, R69, R71, U3, Y1
